File: pcb/sonopi-digi.sch (EAGLE design)
At the start: 10 parts, among them IC1 WM8804, J1 PLT133_T10W, X1 RASPI_BOARD_B+#_SMALL, X2 27MHz/15pF

Commit message: complete PCB design
Parts:
- removed X2: 27MHz/15pF, CRYSTAL3225:CRYSTAL3225HS
- added J2: RASPI_BOARD_B+#_SMALL, raspi-zero:RASPI_BOARD_B+#_SMALL
- X1: value RASPI_BOARD_B+#_SMALL -> 27MHz/15pF; device raspi-zero:RASPI_BOARD_B+#_SMALL -> CRYSTAL3225:CRYSTAL3225HS
Connections:
- net +3V3: now also J2.3V3A, J2.3V3B; no longer X1.3V3A, X1.3V3B
- net BCLK: now also J2.GPIO18; no longer X1.GPIO18
- net DATA: now also J2.GPIO21; no longer X1.GPIO21
- net GND: now also J2.GND_A, J2.GND_B, J2.GND_C, J2.GND_D, J2.GND_E, J2.GND_F, J2.GND_G, J2.GND_H, X1.GND_1, X1.GND_2; no longer X1.GND_A, X1.GND_B, X1.GND_C, X1.GND_D, X1.GND_E, X1.GND_F, X1.GND_G, X1.GND_H, X2.GND_1, X2.GND_2
- net LRCLK: now also J2.GPIO19; no longer X1.GPIO19
- net SCL: now also J2.SCL; no longer X1.SCL
- net SDA: now also J2.SDA; no longer X1.SDA
- net XIN: now also X1.HOT_2; no longer X2.HOT_2
- net XOP: now also X1.HOT_1; no longer X2.HOT_1
Changed lines of the file:
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@@
 </classes>
 <parts>
-<part name="IC1" library="WM8804GEDS_RV" deviceset="WM8804" device=""/>
-<part name="X1" library="raspi-zero" deviceset="RASPI_BOARD_B+#" device="_SMALL" value="RASPI_BOARD_B+#_SMALL"/>
-<part name="J1" library="PLT133_T10W" deviceset="PLT133_T10W" device=""/>
+<part name="IC1" library="WM8804GEDS_RV" library_urn="urn:adsk.eagle:library:9355947" deviceset="WM8804" device="" package3d_urn="urn:adsk.eagle:package:9355950/2"/>
+<part name="J2" library="raspi-zero" library_urn="urn:adsk.eagle:library:9355962" deviceset="RASPI_BOARD_B+#" device="_SMALL" package3d_urn="urn:adsk.eagle:package:9355965/2" value="RASPI_BOARD_B+#_SMALL"/>
+<part name="J1" library="PLT133_T10W" library_urn="urn:adsk.eagle:library:9367061" deviceset="PLT133_T10W" device="" package3d_urn="urn:adsk.eagle:package:9367064/2"/>
 <part name="+3V1" library="supply1" library_urn="urn:adsk.eagle:library:371" deviceset="+3V3" device=""/>
 <part name="GND1" library="supply1" library_urn="urn:adsk.eagle:library:371" deviceset="GND" device=""/>
-<part name="X2" library="CRYSTAL3225" library_urn="urn:adsk.eagle:library:8815235" deviceset="CRYSTAL3225" device="HS" package3d_urn="urn:adsk.eagle:package:8815239/2" value="27MHz/15pF"/>
+<part name="X1" library="CRYSTAL3225" library_urn="urn:adsk.eagle:library:8815235" deviceset="CRYSTAL3225" device="HS" package3d_urn="urn:adsk.eagle:package:8815239/2" value="27MHz/15pF"/>
 <part name="C1" library="gen-discrete2" library_urn="urn:adsk.eagle:library:7031920" deviceset="CAPACITOR" device="1608" package3d_urn="urn:adsk.eagle:package:5494249/3" value="1u"/>
 <part name="C2" library="gen-discrete2" library_urn="urn:adsk.eagle:library:7031920" deviceset="CAPACITOR" device="1608" package3d_urn="urn:adsk.eagle:package:5494249/3" value="0.1u"/>
@@
 <attribute name="VALUE" x="127.508" y="69.088" size="1.778" layer="96" align="center-left"/>
 </instance>
-<instance part="X1" gate="G$1" x="40.64" y="60.96" smashed="yes"/>
+<instance part="J2" gate="G$1" x="40.64" y="60.96" smashed="yes"/>
 <instance part="J1" gate="G$1" x="175.26" y="10.16" smashed="yes">
 <attribute name="NAME" x="189.23" y="15.24" size="1.778" layer="95" align="center"/>
@@
 <attribute name="VALUE" x="63.5" y="27.94" size="1.778" layer="96"/>
 </instance>
-<instance part="X2" gate="G$1" x="142.24" y="58.42" smashed="yes">
+<instance part="X1" gate="G$1" x="142.24" y="58.42" smashed="yes">
 <attribute name="NAME" x="141.986" y="66.04" size="1.778" layer="95" align="center"/>
 <attribute name="VALUE" x="141.732" y="62.992" size="1.778" layer="96" align="center"/>
@@
 <net name="BCLK" class="0">
 <segment>
-<pinref part="X1" gate="G$1" pin="GPIO18"/>
+<pinref part="J2" gate="G$1" pin="GPIO18"/>
 <wire x1="25.4" y1="73.66" x2="12.7" y2="73.66" width="0.1524" layer="91"/>
 <label x="12.7" y="73.66" size="1.778" layer="95"/>
@@
 <net name="SCL" class="0">
 <segment>
-<pinref part="X1" gate="G$1" pin="SCL"/>
+<pinref part="J2" gate="G$1" pin="SCL"/>
 <wire x1="25.4" y1="27.94" x2="12.7" y2="27.94" width="0.1524" layer="91"/>
 <label x="12.7" y="27.94" size="1.778" layer="95"/>
@@
 <net name="SDA" class="0">
 <segment>
-<pinref part="X1" gate="G$1" pin="SDA"/>
+<pinref part="J2" gate="G$1" pin="SDA"/>
 <wire x1="25.4" y1="25.4" x2="12.7" y2="25.4" width="0.1524" layer="91"/>
 <label x="12.7" y="25.4" size="1.778" layer="95"/>
@@
 <net name="+3V3" class="0">
 <segment>
-<pinref part="X1" gate="G$1" pin="3V3A"/>
+<pinref part="J2" gate="G$1" pin="3V3A"/>
 <pinref part="+3V1" gate="G$1" pin="+3V3"/>
 <wire x1="45.72" y1="88.9" x2="45.72" y2="91.44" width="0.1524" layer="91"/>
-<pinref part="X1" gate="G$1" pin="3V3B"/>
+<pinref part="J2" gate="G$1" pin="3V3B"/>
 <wire x1="45.72" y1="91.44" x2="45.72" y2="93.98" width="0.1524" layer="91"/>
 <wire x1="48.26" y1="88.9" x2="48.26" y2="91.44" width="0.1524" layer="91"/>
@@
 <net name="GND" class="0">
 <segment>
-<pinref part="X1" gate="G$1" pin="GND_B"/>
+<pinref part="J2" gate="G$1" pin="GND_B"/>
 <wire x1="55.88" y1="50.8" x2="66.04" y2="50.8" width="0.1524" layer="91"/>
 <pinref part="GND1" gate="1" pin="GND"/>
 <wire x1="66.04" y1="50.8" x2="66.04" y2="48.26" width="0.1524" layer="91"/>
-<pinref part="X1" gate="G$1" pin="GND_E"/>
+<pinref part="J2" gate="G$1" pin="GND_E"/>
 <wire x1="66.04" y1="48.26" x2="66.04" y2="45.72" width="0.1524" layer="91"/>
 <wire x1="66.04" y1="45.72" x2="66.04" y2="43.18" width="0.1524" layer="91"/>
@@
 <wire x1="55.88" y1="43.18" x2="66.04" y2="43.18" width="0.1524" layer="91"/>
 <junction x="66.04" y="43.18"/>
-<pinref part="X1" gate="G$1" pin="GND_H"/>
+<pinref part="J2" gate="G$1" pin="GND_H"/>
 <wire x1="55.88" y1="35.56" x2="66.04" y2="35.56" width="0.1524" layer="91"/>
 <junction x="66.04" y="35.56"/>
-<pinref part="X1" gate="G$1" pin="GND_A"/>
+<pinref part="J2" gate="G$1" pin="GND_A"/>
 <wire x1="55.88" y1="53.34" x2="66.04" y2="53.34" width="0.1524" layer="91"/>
 <wire x1="66.04" y1="53.34" x2="66.04" y2="50.8" width="0.1524" layer="91"/>
 <junction x="66.04" y="50.8"/>
-<pinref part="X1" gate="G$1" pin="GND_G"/>
+<pinref part="J2" gate="G$1" pin="GND_G"/>
 <wire x1="55.88" y1="38.1" x2="66.04" y2="38.1" width="0.1524" layer="91"/>
 <junction x="66.04" y="38.1"/>
-<pinref part="X1" gate="G$1" pin="GND_C"/>
+<pinref part="J2" gate="G$1" pin="GND_C"/>
 <wire x1="55.88" y1="48.26" x2="66.04" y2="48.26" width="0.1524" layer="91"/>
 <junction x="66.04" y="48.26"/>
-<pinref part="X1" gate="G$1" pin="GND_D"/>
+<pinref part="J2" gate="G$1" pin="GND_D"/>
 <wire x1="55.88" y1="45.72" x2="66.04" y2="45.72" width="0.1524" layer="91"/>
 <junction x="66.04" y="45.72"/>
-<pinref part="X1" gate="G$1" pin="GND_F"/>
+<pinref part="J2" gate="G$1" pin="GND_F"/>
 <wire x1="55.88" y1="40.64" x2="66.04" y2="40.64" width="0.1524" layer="91"/>
 <junction x="66.04" y="40.64"/>
@@
 <wire x1="144.78" y1="45.72" x2="154.94" y2="45.72" width="0.1524" layer="91"/>
 <wire x1="154.94" y1="45.72" x2="154.94" y2="50.8" width="0.1524" layer="91"/>
-<pinref part="X2" gate="G$1" pin="GND_1"/>
+<pinref part="X1" gate="G$1" pin="GND_1"/>
 <wire x1="139.7" y1="48.26" x2="139.7" y2="45.72" width="0.1524" layer="91"/>
 <junction x="139.7" y="45.72"/>
-<pinref part="X2" gate="G$1" pin="GND_2"/>
+<pinref part="X1" gate="G$1" pin="GND_2"/>
 <wire x1="144.78" y1="48.26" x2="144.78" y2="45.72" width="0.1524" layer="91"/>
 <junction x="144.78" y="45.72"/>
@@
 <pinref part="IC1" gate="G$1" pin="XOP"/>
 <wire x1="121.92" y1="73.66" x2="119.38" y2="73.66" width="0.1524" layer="91"/>
-<pinref part="X2" gate="G$1" pin="HOT_1"/>
+<pinref part="X1" gate="G$1" pin="HOT_1"/>
 <wire x1="119.38" y1="73.66" x2="119.38" y2="58.42" width="0.1524" layer="91"/>
 <wire x1="119.38" y1="58.42" x2="127" y2="58.42" width="0.1524" layer="91"/>
@@
 <pinref part="IC1" gate="G$1" pin="XIN"/>
 <wire x1="162.56" y1="73.66" x2="165.1" y2="73.66" width="0.1524" layer="91"/>
-<pinref part="X2" gate="G$1" pin="HOT_2"/>
+<pinref part="X1" gate="G$1" pin="HOT_2"/>
 <wire x1="165.1" y1="73.66" x2="165.1" y2="58.42" width="0.1524" layer="91"/>
 <wire x1="165.1" y1="58.42" x2="154.94" y2="58.42" width="0.1524" layer="91"/>
@@
 </segment>
 <segment>
-<pinref part="X1" gate="G$1" pin="GPIO21"/>
+<pinref part="J2" gate="G$1" pin="GPIO21"/>
 <wire x1="25.4" y1="33.02" x2="12.7" y2="33.02" width="0.1524" layer="91"/>
 <label x="12.7" y="33.02" size="1.778" layer="95"/>
@@
 <net name="LRCLK" class="0">
 <segment>
-<pinref part="X1" gate="G$1" pin="GPIO19"/>
+<pinref part="J2" gate="G$1" pin="GPIO19"/>
 <wire x1="25.4" y1="43.18" x2="12.7" y2="43.18" width="0.1524" layer="91"/>
 <label x="12.7" y="43.18" size="1.778" layer="95"/>

Commit message: improve wiring
Connections:
- new net VDD: C2.1, IC1.DVDD, J2.3V3B
- net +3V3: no longer C2.1, IC1.DVDD, J2.3V3B
Changed lines of the file:
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@@
 <part name="GND2" library="supply1" library_urn="urn:adsk.eagle:library:371" deviceset="GND" device=""/>
 <part name="GND3" library="supply1" library_urn="urn:adsk.eagle:library:371" deviceset="GND" device=""/>
-<part name="+3V3" library="supply1" library_urn="urn:adsk.eagle:library:371" deviceset="+3V3" device=""/>
 <part name="GND4" library="supply1" library_urn="urn:adsk.eagle:library:371" deviceset="GND" device=""/>
 <part name="C5" library="gen-discrete2" library_urn="urn:adsk.eagle:library:7031920" deviceset="CAPACITOR" device="1608" package3d_urn="urn:adsk.eagle:package:5494249/3" value="0.1u"/>
@@
 <part name="+3V5" library="supply1" library_urn="urn:adsk.eagle:library:371" deviceset="+3V3" device=""/>
 <part name="GND6" library="supply1" library_urn="urn:adsk.eagle:library:371" deviceset="GND" device=""/>
+<part name="VDD1" library="supply1" library_urn="urn:adsk.eagle:library:371" deviceset="VDD" device=""/>
+<part name="VDD2" library="supply1" library_urn="urn:adsk.eagle:library:371" deviceset="VDD" device=""/>
 </parts>
 <sheets>
@@
 <attribute name="VALUE" x="172.72" y="91.44" size="1.778" layer="96"/>
 </instance>
-<instance part="+3V3" gate="G$1" x="175.26" y="114.3" smashed="yes">
-<attribute name="VALUE" x="171.704" y="115.316" size="1.778" layer="96"/>
-</instance>
 <instance part="GND4" gate="1" x="142.24" y="40.64" smashed="yes">
 <attribute name="VALUE" x="139.7" y="38.1" size="1.778" layer="96"/>
@@
 <instance part="GND6" gate="1" x="99.06" y="15.24" smashed="yes">
 <attribute name="VALUE" x="96.52" y="12.7" size="1.778" layer="96"/>
+</instance>
+<instance part="VDD1" gate="G$1" x="53.34" y="96.52" smashed="yes">
+<attribute name="VALUE" x="51.054" y="98.298" size="1.778" layer="96"/>
+</instance>
+<instance part="VDD2" gate="G$1" x="175.26" y="114.3" smashed="yes">
+<attribute name="VALUE" x="172.974" y="116.078" size="1.778" layer="96"/>
 </instance>
 </instances>
@@
 <pinref part="J2" gate="G$1" pin="3V3A"/>
 <pinref part="+3V1" gate="G$1" pin="+3V3"/>
-<wire x1="45.72" y1="88.9" x2="45.72" y2="91.44" width="0.1524" layer="91"/>
-<pinref part="J2" gate="G$1" pin="3V3B"/>
-<wire x1="45.72" y1="91.44" x2="45.72" y2="93.98" width="0.1524" layer="91"/>
-<wire x1="48.26" y1="88.9" x2="48.26" y2="91.44" width="0.1524" layer="91"/>
-<wire x1="48.26" y1="91.44" x2="45.72" y2="91.44" width="0.1524" layer="91"/>
-<junction x="45.72" y="91.44"/>
+<wire x1="45.72" y1="88.9" x2="45.72" y2="93.98" width="0.1524" layer="91"/>
 </segment>
 <segment>
@@
 <wire x1="99.06" y1="83.82" x2="99.06" y2="81.28" width="0.1524" layer="91"/>
 <junction x="99.06" y="81.28"/>
-</segment>
-<segment>
-<pinref part="IC1" gate="G$1" pin="DVDD"/>
-<wire x1="162.56" y1="93.98" x2="165.1" y2="93.98" width="0.1524" layer="91"/>
-<wire x1="165.1" y1="93.98" x2="165.1" y2="109.22" width="0.1524" layer="91"/>
-<wire x1="165.1" y1="109.22" x2="175.26" y2="109.22" width="0.1524" layer="91"/>
-<pinref part="C2" gate="G$1" pin="1"/>
-<wire x1="175.26" y1="109.22" x2="175.26" y2="106.68" width="0.1524" layer="91"/>
-<pinref part="+3V3" gate="G$1" pin="+3V3"/>
-<wire x1="175.26" y1="109.22" x2="175.26" y2="111.76" width="0.1524" layer="91"/>
-<junction x="175.26" y="109.22"/>
 </segment>
 <segment>
@@
 </segment>
 </net>
+<net name="VDD" class="0">
+<segment>
+<pinref part="J2" gate="G$1" pin="3V3B"/>
+<wire x1="48.26" y1="88.9" x2="48.26" y2="91.44" width="0.1524" layer="91"/>
+<wire x1="48.26" y1="91.44" x2="53.34" y2="91.44" width="0.1524" layer="91"/>
+<pinref part="VDD1" gate="G$1" pin="VDD"/>
+<wire x1="53.34" y1="91.44" x2="53.34" y2="93.98" width="0.1524" layer="91"/>
+</segment>
+<segment>
+<pinref part="IC1" gate="G$1" pin="DVDD"/>
+<wire x1="162.56" y1="93.98" x2="165.1" y2="93.98" width="0.1524" layer="91"/>
+<wire x1="165.1" y1="93.98" x2="165.1" y2="109.22" width="0.1524" layer="91"/>
+<wire x1="165.1" y1="109.22" x2="175.26" y2="109.22" width="0.1524" layer="91"/>
+<pinref part="C2" gate="G$1" pin="1"/>
+<wire x1="175.26" y1="109.22" x2="175.26" y2="106.68" width="0.1524" layer="91"/>
+<pinref part="VDD2" gate="G$1" pin="VDD"/>
+<wire x1="175.26" y1="111.76" x2="175.26" y2="109.22" width="0.1524" layer="91"/>
+<junction x="175.26" y="109.22"/>
+</segment>
+</net>
